File: test/fixtures/benchmark_projects/fail_bad_decoupling_placement/demo.kicad_sch (KiCad schematic)
At the start: 0 parts

Commit message: test(fixtures): clean up and fix benchmark project fixtures
- Remove 4 empty kicad10_* stub projects (kicad10_variants,
  kicad10_timedomain, kicad10_custom_drc, kicad10_design_blocks)
  that had no schematic/PCB content and were not referenced by any test
- Remove stray demo.kicad_prl from fail_bad_decoupling_placement
- Fix 3 fail_* projects whose schematics were empty while PCBs had
  content (fail_bad_decoupling_placement, fail_dfm_edge_clearance,
  fail_sensor_cluster_spread): add matching component symbols
- Fix 3 fail_* projects whose PCBs were empty while schematics had
  content (fail_label_only_schematic, fail_sismosmart_like_hierarchy,
  fail_sismosmart_like_label_only): add matching footprints

All 10 remaining fixtures now have consistent schematic + PCB content
that matches their intended failure scenario.
Parts:
- added C1: 100n, Capacitor_SMD:C_0603_1608Metric, symbol Device:C
- added U1: ATmega328P, Package_QFP:TQFP-32_7x7mm_P0.8mm, symbol MCU_Microchip_ATmega:ATmega328P-AU
Changed lines of the file:
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@@
   (generator "pytest")
   (paper "A4")
+  (symbol
+    (lib_id "MCU_Microchip_ATmega:ATmega328P-AU")
+    (at 10.16 10.16 0)
+    (unit 1)
+    (property "Reference" "U1" (at 10.16 5.08 0))
+    (property "Value" "ATmega328P" (at 10.16 15.24 0))
+    (property "Footprint" "Package_QFP:TQFP-32_7x7mm_P0.8mm" (at 10.16 17.78 0))
+  )
+  (symbol
+    (lib_id "Device:C")
+    (at 30.48 10.16 0)
+    (unit 1)
+    (property "Reference" "C1" (at 30.48 7.62 0))
+    (property "Value" "100n" (at 30.48 12.7 0))
+    (property "Footprint" "Capacitor_SMD:C_0603_1608Metric" (at 30.48 15.24 0))
+  )
+  (global_label "VCC" (shape input) (at 10.16 2.54 0) (effects (font (size 1.27 1.27))))
+  (global_label "GND" (shape bidirectional) (at 30.48 17.78 0) (effects (font (size 1.27 1.27))))
   (sheet_instances
     (path "/" (page "1"))
