File: test/fixtures/benchmark_projects/fail_dfm_edge_clearance/demo.kicad_sch (KiCad schematic)
At the start: 0 parts

Commit message: test(fixtures): clean up and fix benchmark project fixtures
- Remove 4 empty kicad10_* stub projects (kicad10_variants,
  kicad10_timedomain, kicad10_custom_drc, kicad10_design_blocks)
  that had no schematic/PCB content and were not referenced by any test
- Remove stray demo.kicad_prl from fail_bad_decoupling_placement
- Fix 3 fail_* projects whose schematics were empty while PCBs had
  content (fail_bad_decoupling_placement, fail_dfm_edge_clearance,
  fail_sensor_cluster_spread): add matching component symbols
- Fix 3 fail_* projects whose PCBs were empty while schematics had
  content (fail_label_only_schematic, fail_sismosmart_like_hierarchy,
  fail_sismosmart_like_label_only): add matching footprints

All 10 remaining fixtures now have consistent schematic + PCB content
that matches their intended failure scenario.
Parts:
- added J1: EdgeTooClose, Connector_Generic:Conn_01x02, symbol Connector_Generic:Conn_01x02
Changed lines of the file:
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@@
   (generator "pytest")
   (paper "A4")
+  (symbol
+    (lib_id "Connector_Generic:Conn_01x02")
+    (at 10.16 10.16 0)
+    (unit 1)
+    (property "Reference" "J1" (at 10.16 7.62 0))
+    (property "Value" "EdgeTooClose" (at 10.16 12.7 0))
+    (property "Footprint" "Connector_Generic:Conn_01x02" (at 10.16 15.24 0))
+  )
+  (global_label "SIG" (shape input) (at 7.62 10.16 0) (effects (font (size 1.27 1.27))))
+  (global_label "GND" (shape bidirectional) (at 7.62 12.7 0) (effects (font (size 1.27 1.27))))
   (sheet_instances
     (path "/" (page "1"))
