File: test/fixtures/benchmark_projects/fail_sismosmart_like_label_only/demo.kicad_pcb (KiCad board)
At the start: 0 parts

Commit message: test(fixtures): clean up and fix benchmark project fixtures
- Remove 4 empty kicad10_* stub projects (kicad10_variants,
  kicad10_timedomain, kicad10_custom_drc, kicad10_design_blocks)
  that had no schematic/PCB content and were not referenced by any test
- Remove stray demo.kicad_prl from fail_bad_decoupling_placement
- Fix 3 fail_* projects whose schematics were empty while PCBs had
  content (fail_bad_decoupling_placement, fail_dfm_edge_clearance,
  fail_sensor_cluster_spread): add matching component symbols
- Fix 3 fail_* projects whose PCBs were empty while schematics had
  content (fail_label_only_schematic, fail_sismosmart_like_hierarchy,
  fail_sismosmart_like_label_only): add matching footprints

All 10 remaining fixtures now have consistent schematic + PCB content
that matches their intended failure scenario.
Parts:
- added J1: USB_C, Connector_USB:USB_C_Receptacle_GCT_USB4110, F.Cu at (5.00, 15.0)
- added U1: ESP32-S3-WROOM-1, RF_Module:ESP32-S3-WROOM-1, F.Cu at (35.0, 25.0)
- added U8: AP2112K-3.3, Package_TO_SOT_SMD:SOT-23-5, F.Cu at (10.0, 40.0)
Other:
- board outline added: 70 x 50 mm
Changed lines of the file:
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@@
-(kicad_pcb)
+(kicad_pcb
+  (version 20250216)
+  (generator "pytest")
+  (gr_rect (start 0 0) (end 70 50) (stroke (width 0.05) (type solid)) (fill no) (layer "Edge.Cuts"))
+  (footprint "RF_Module:ESP32-S3-WROOM-1"
+    (layer "F.Cu")
+    (at 35 25 0)
+    (property "Reference" "U1" (at 0 0 0) (layer "F.SilkS"))
+    (property "Value" "ESP32-S3-WROOM-1" (at 0 9 0) (layer "F.Fab"))
+    (fp_rect (start -9 -6.5) (end 9 9) (stroke (width 0.05) (type solid)) (fill no) (layer "F.CrtYd"))
+  )
+  (footprint "Package_TO_SOT_SMD:SOT-23-5"
+    (layer "F.Cu")
+    (at 10 40 0)
+    (property "Reference" "U8" (at 0 0 0) (layer "F.SilkS"))
+    (property "Value" "AP2112K-3.3" (at 0 2.5 0) (layer "F.Fab"))
+    (fp_rect (start -1.8 -1.5) (end 1.8 2) (stroke (width 0.05) (type solid)) (fill no) (layer "F.CrtYd"))
+  )
+  (footprint "Connector_USB:USB_C_Receptacle_GCT_USB4110"
+    (layer "F.Cu")
+    (at 5 15 0)
+    (property "Reference" "J1" (at 0 0 0) (layer "F.SilkS"))
+    (property "Value" "USB_C" (at 0 4 0) (layer "F.Fab"))
+    (fp_rect (start -5 -2) (end 5 4.5) (stroke (width 0.05) (type solid)) (fill no) (layer "F.CrtYd"))
+  )
+)
